Commit message: corridor_description: low lateral wheel friction (mu2 0.15 along fdir1) so the skid steer can turn (#19)
Measured in Gazebo before: 1.0 rad/s commanded in place gave 0.22 rad/s; the vehicle overshot every corner.

Co-Authored-By: Claude Fable 5.1 <noreply@anthropic.com>

File: ws/src/corridor_description/urdf/ugv.gazebo.xacro (robot description, xacro)
@@ -4,4 +4,18 @@
        Topic names are gz-side; corridor_gz/config/bridge.yaml maps them to ROS. -->
   <xacro:macro name="ugv_gazebo" params="prefix ns">
+    <!-- Skid steer: full lateral grip on four wheels 0.8 m apart lets the vehicle turn at a quarter of
+         the commanded rate (measured 0.22 rad/s for 1.0). Low mu2 across the rolling direction lets the
+         wheels slide sideways as rubber on gravel does. -->
+    <xacro:macro name="wheel_friction" params="name">
+      <gazebo reference="${prefix}${name}_wheel">
+        <collision>
+          <surface><friction><ode><mu>1.0</mu><mu2>0.15</mu2><fdir1>1 0 0</fdir1></ode></friction></surface>
+        </collision>
+      </gazebo>
+    </xacro:macro>
+    <xacro:wheel_friction name="front_left"/>
+    <xacro:wheel_friction name="front_right"/>
+    <xacro:wheel_friction name="rear_left"/>
+    <xacro:wheel_friction name="rear_right"/>
     <gazebo reference="${prefix}lidar_link">
       <sensor name="lidar" type="gpu_lidar">
